File: standard_puzzle_module/standard_puzzle_box.kicad_pcb (KiCad board)
At the start: 2 copper layers, 76 parts, among them U1 ESP32-C3-DevKitM-1

Commit message: fix: block reverse current in BO block rather than lead it to gnd
Parts:
- moved Q_BO3 94.3 mm to (327.9, 103.0)
- moved CC_BO3 94.3 mm to (317.5, 102.5)
- moved U_BO3 94.3 mm to (317.2, 94.2)
- moved J_BO1 89.5 mm to (329.9, 17.0)
- moved CP_BO1 89.5 mm to (342.1, 16.5)
- moved D_BO1 89.5 mm to (340.3, 25.1)
- moved R_BO5 89.5 mm to (301.4, 20.5)
- moved R_BO6 89.5 mm to (301.5, 26.5)
- moved Q_BO1 89.5 mm to (329.4, 27.5)
- moved CC_BO1 45.3 mm to (308.0, 116.0)
- moved U_BO1 35.3 mm to (300.7, 104.2)
- moved J_BI3 24.5 mm to (55.5, 168.2)
- moved J_BI4 23.3 mm to (29.5, 168.2)
- moved D_BI3 14.6 mm to (46.3, 156.5), turned to 90 degrees
- moved D_TVSP1 13.7 mm to (175.3, 120.0)
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
Commit message: feat: creating backup and trying to fix broken project state
Parts:
- moved FUSE1 35.4 mm to (148.5, 130.0)
- moved CC_PI1 35.4 mm to (157.9, 116.5)
- moved CC_PO1 35.4 mm to (157.4, 97.5)
- moved CP_PI1 35.4 mm to (157.9, 128.0)
- moved CP_PO1 35.4 mm to (159.9, 102.5)
- moved DCREG1 35.4 mm to (150.4, 103.5)
- moved D_SCHP1 35.4 mm to (150.4, 109.9)
- moved J_PWR1 31.7 mm to (151.9, 148.5)
Changed lines of the file:
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@@
 	(footprint "Converter_DCDC:Converter_DCDC_RECOM_R-78E-0.5_THT"
 		(layer "F.Cu")
-		(at 136.5 136 90)
+		(at 150.42 103.5 90)
 		(descr "DCDC-Converter, RECOM, RECOM_R-78E-0.5, SIP-3, pitch 2.54mm, package size 11.6x8.5x10.4mm^3, https://www.recom-power.com/pdf/Innoline/R-78Exx-0.5.pdf")
 		(tags "dc-dc recom buck sip-3 pitch 2.54mm")
@@
 	(footprint "TerminalBlock_Phoenix:TerminalBlock_Phoenix_MKDS-1,5-2-5.08_1x02_P5.08mm_Horizontal"
 		(layer "F.Cu")
-		(at 134.5 175)
+		(at 151.92 148.5)
 		(descr "Terminal Block Phoenix MKDS-1,5-2-5.08, 2 pins, pitch 5.08mm, size 10.2x9.8mm, drill diameter 1.3mm, pad diameter 2.6mm, http://www.farnell.com/datasheets/100425.pdf")
 		(tags "THT Terminal Block Phoenix MKDS-1,5-2-5.08 pitch 5.08mm size 10.2x9.8mm drill 1.3mm pad 2.6mm")
@@
 		)
 		(property "Value" "100nF"
-			(at 48.63 87.69 0)
+			(at 62.55 55.19 0)
 			(layer "F.Fab")
 			(effects
@@
 	(footprint "Capacitor_THT:CP_Radial_D6.3mm_P2.50mm"
 		(layer "F.Cu")
-		(at 146 135 -90)
+		(at 159.92 102.5 -90)
 		(descr "CP, Radial series, Radial, pin pitch=2.50mm, diameter=6.3mm, height=7mm, Electrolytic Capacitor")
 		(tags "CP Radial series Radial pin pitch 2.50mm diameter 6.3mm height 7mm Electrolytic Capacitor")
@@
 	(footprint "Capacitor_THT:C_Disc_D5.0mm_W2.5mm_P5.00mm"
 		(layer "F.Cu")
-		(at 143.5 130)
+		(at 157.42 97.5)
 		(descr "C, Disc series, Radial, pin pitch=5.00mm, diameter*width=5*2.5mm^2, Capacitor, http://cdn-reichelt.de/documents/datenblatt/B300/DS_KERKO_TC.pdf")
 		(tags "C Disc series Radial pin pitch 5.00mm diameter 5mm width 2.5mm Capacitor")
@@
 	(footprint "Fuse:Fuse_BelFuse_0ZRE0040FF_L11.5mm_W3.8mm"
 		(layer "F.Cu")
-		(at 134.6 162.5 90)
+		(at 148.52 130 90)
 		(descr "Fuse 0ZRE0040FF, BelFuse, Radial Leaded PTC,https://www.belfuse.com/resources/datasheets/circuitprotection/ds-cp-0zre-series.pdf")
 		(tags "0ZRE BelFuse radial PTC")
@@
 	(footprint "Capacitor_THT:C_Disc_D5.0mm_W2.5mm_P5.00mm"
 		(layer "F.Cu")
-		(at 144 149)
+		(at 157.92 116.5)
 		(descr "C, Disc series, Radial, pin pitch=5.00mm, diameter*width=5*2.5mm^2, Capacitor, http://cdn-reichelt.de/documents/datenblatt/B300/DS_KERKO_TC.pdf")
 		(tags "C Disc series Radial pin pitch 5.00mm diameter 5mm width 2.5mm Capacitor")
@@
 	(footprint "Capacitor_THT:CP_Radial_D10.0mm_P5.00mm"
 		(layer "F.Cu")
-		(at 144 160.5)
+		(at 157.92 128)
 		(descr "CP, Radial series, Radial, pin pitch=5.00mm, diameter=10mm, height=16mm, Electrolytic Capacitor")
 		(tags "CP Radial series Radial pin pitch 5.00mm diameter 10mm height 16mm Electrolytic Capacitor")
@@
 	(footprint "Diode_THT:D_DO-35_SOD27_P7.62mm_Horizontal"
 		(layer "F.Cu")
-		(at 136.5 142.38 -90)
+		(at 150.42 109.88 -90)
 		(descr "Diode, DO-35_SOD27 series, Axial, Horizontal, pin pitch=7.62mm, length*diameter=4*2mm^2, http://www.diodes.com/_files/packages/DO-35.pdf")
 		(tags "Diode DO-35_SOD27 series Axial Horizontal pin pitch 7.62mm  length 4mm diameter 2mm")
