File: standard_puzzle_module/boolean_output.kicad_sch (KiCad schematic)
At the start: 8 parts, among them J7 Screw_Terminal_01x02, Q3 IRLZ44N, U7 PC817

Commit message: feat: unscrew git tracking
Changed lines of the file:
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@@
+	)
+	(junction
+		(at 104.14 90.17)
+		(diameter 0)
+		(color 0 0 0 0)
 	)
 	(junction
@@
 	(wire
 		(pts
+			(xy 104.14 90.17) (xy 104.14 92.71)
+		)
+		(stroke
+			(width 0)
+			(type default)
+		)
+	)
+	(wire
+		(pts
 			(xy 116.84 96.52) (xy 120.65 96.52)
 		)
@@
 	(wire
 		(pts
-			(xy 104.14 86.36) (xy 104.14 92.71)
+			(xy 104.14 86.36) (xy 104.14 90.17)
 		)
 		(stroke
@@
 		(pts
 			(xy 154.94 106.68) (xy 154.94 109.22)
+		)
+		(stroke
+			(width 0)
+			(type default)
+		)
+	)
+	(wire
+		(pts
+			(xy 99.06 90.17) (xy 104.14 90.17)
 		)
 		(stroke
@@
 				(justify left)
 			)
+		)
+	)
+	(hierarchical_label "out"
+		(shape input)
+		(at 99.06 90.17 180)
+		(effects
+			(font
+				(size 1.27 1.27)
+			)
+			(justify right)
 		)
 	)
@@
 		(instances
 			(project "standard_puzzle_box"
+				(path "/13314f97-080e-4924-a8fe-b4d224920625/05a99c97-6240-4e5e-b6a9-a36dfb628c26"
+					(reference "#PWR079")
+					(unit 1)
+				)
 				(path "/13314f97-080e-4924-a8fe-b4d224920625/a03c39d6-6910-42d9-b21d-b8f6aa6403fb"
 					(reference "#PWR034")
+					(unit 1)
+				)
+				(path "/13314f97-080e-4924-a8fe-b4d224920625/d25a32d7-442e-482e-90f8-47542d85b960"
+					(reference "#PWR074")
 					(unit 1)
 				)
@@
 		(instances
 			(project "standard_puzzle_box"
+				(path "/13314f97-080e-4924-a8fe-b4d224920625/05a99c97-6240-4e5e-b6a9-a36dfb628c26"
+					(reference "#PWR082")
+					(unit 1)
+				)
 				(path "/13314f97-080e-4924-a8fe-b4d224920625/a03c39d6-6910-42d9-b21d-b8f6aa6403fb"
 					(reference "#PWR037")
+					(unit 1)
+				)
+				(path "/13314f97-080e-4924-a8fe-b4d224920625/d25a32d7-442e-482e-90f8-47542d85b960"
+					(reference "#PWR077")
 					(unit 1)
 				)
@@
 		(instances
 			(project "standard_puzzle_box"
+				(path "/13314f97-080e-4924-a8fe-b4d224920625/05a99c97-6240-4e5e-b6a9-a36dfb628c26"
+					(reference "D1flyback4")
+					(unit 1)
+				)
 				(path "/13314f97-080e-4924-a8fe-b4d224920625/a03c39d6-6910-42d9-b21d-b8f6aa6403fb"
 					(reference "D1flyback2")
+					(unit 1)
+				)
+				(path "/13314f97-080e-4924-a8fe-b4d224920625/d25a32d7-442e-482e-90f8-47542d85b960"
+					(reference "D1flyback3")
 					(unit 1)
 				)
@@
 		(instances
 			(project "standard_puzzle_box"
+				(path "/13314f97-080e-4924-a8fe-b4d224920625/05a99c97-6240-4e5e-b6a9-a36dfb628c26"
+					(reference "C24")
+					(unit 1)
+				)
 				(path "/13314f97-080e-4924-a8fe-b4d224920625/a03c39d6-6910-42d9-b21d-b8f6aa6403fb"
 					(reference "C11")
+					(unit 1)
+				)
+				(path "/13314f97-080e-4924-a8fe-b4d224920625/d25a32d7-442e-482e-90f8-47542d85b960"
+					(reference "C22")
 					(unit 1)
 				)
@@
 		(instances
 			(project "standard_puzzle_box"
+				(path "/13314f97-080e-4924-a8fe-b4d224920625/05a99c97-6240-4e5e-b6a9-a36dfb628c26"
+					(reference "U14")
+					(unit 1)
+				)
 				(path "/13314f97-080e-4924-a8fe-b4d224920625/a03c39d6-6910-42d9-b21d-b8f6aa6403fb"
 					(reference "U7")
+					(unit 1)
+				)
+				(path "/13314f97-080e-4924-a8fe-b4d224920625/d25a32d7-442e-482e-90f8-47542d85b960"
+					(reference "U13")
 					(unit 1)
 				)
@@
 		(instances
 			(project "standard_puzzle_box"
+				(path "/13314f97-080e-4924-a8fe-b4d224920625/05a99c97-6240-4e5e-b6a9-a36dfb628c26"
+					(reference "R27")
+					(unit 1)
+				)
 				(path "/13314f97-080e-4924-a8fe-b4d224920625/a03c39d6-6910-42d9-b21d-b8f6aa6403fb"
 					(reference "R9")
+					(unit 1)
+				)
+				(path "/13314f97-080e-4924-a8fe-b4d224920625/d25a32d7-442e-482e-90f8-47542d85b960"
+					(reference "R14")
 					(unit 1)
 				)
@@
 		(instances
 			(project "standard_puzzle_box"
+				(path "/13314f97-080e-4924-a8fe-b4d224920625/05a99c97-6240-4e5e-b6a9-a36dfb628c26"
+					(reference "#PWR078")
+					(unit 1)
+				)
 				(path "/13314f97-080e-4924-a8fe-b4d224920625/a03c39d6-6910-42d9-b21d-b8f6aa6403fb"
 					(reference "#PWR033")
+					(unit 1)
+				)
+				(path "/13314f97-080e-4924-a8fe-b4d224920625/d25a32d7-442e-482e-90f8-47542d85b960"
+					(reference "#PWR073")
 					(unit 1)
 				)
@@
 		(instances
 			(project "standard_puzzle_box"
+				(path "/13314f97-080e-4924-a8fe-b4d224920625/05a99c97-6240-4e5e-b6a9-a36dfb628c26"
+					(reference "C23")
+					(unit 1)
+				)
 				(path "/13314f97-080e-4924-a8fe-b4d224920625/a03c39d6-6910-42d9-b21d-b8f6aa6403fb"
 					(reference "C10")
+					(unit 1)
+				)
+				(path "/13314f97-080e-4924-a8fe-b4d224920625/d25a32d7-442e-482e-90f8-47542d85b960"
+					(reference "C21")
 					(unit 1)
 				)
@@
 		(instances
 			(project "standard_puzzle_box"
+				(path "/13314f97-080e-4924-a8fe-b4d224920625/05a99c97-6240-4e5e-b6a9-a36dfb628c26"
+					(reference "Q5")
+					(unit 1)
+				)
 				(path "/13314f97-080e-4924-a8fe-b4d224920625/a03c39d6-6910-42d9-b21d-b8f6aa6403fb"
 					(reference "Q3")
+					(unit 1)
+				)
+				(path "/13314f97-080e-4924-a8fe-b4d224920625/d25a32d7-442e-482e-90f8-47542d85b960"
+					(reference "Q4")
 					(unit 1)
 				)
@@
 		(instances
 			(project "standard_puzzle_box"
+				(path "/13314f97-080e-4924-a8fe-b4d224920625/05a99c97-6240-4e5e-b6a9-a36dfb628c26"
+					(reference "#PWR080")
+					(unit 1)
+				)
 				(path "/13314f97-080e-4924-a8fe-b4d224920625/a03c39d6-6910-42d9-b21d-b8f6aa6403fb"
 					(reference "#PWR035")
+					(unit 1)
+				)
+				(path "/13314f97-080e-4924-a8fe-b4d224920625/d25a32d7-442e-482e-90f8-47542d85b960"
+					(reference "#PWR075")
 					(unit 1)
 				)
@@
 		(instances
 			(project "standard_puzzle_box"
+				(path "/13314f97-080e-4924-a8fe-b4d224920625/05a99c97-6240-4e5e-b6a9-a36dfb628c26"
+					(reference "R28")
+					(unit 1)
+				)
 				(path "/13314f97-080e-4924-a8fe-b4d224920625/a03c39d6-6910-42d9-b21d-b8f6aa6403fb"
 					(reference "R16")
+					(unit 1)
+				)
+				(path "/13314f97-080e-4924-a8fe-b4d224920625/d25a32d7-442e-482e-90f8-47542d85b960"
+					(reference "R26")
 					(unit 1)
 				)
@@
 		(instances
 			(project "standard_puzzle_box"
+				(path "/13314f97-080e-4924-a8fe-b4d224920625/05a99c97-6240-4e5e-b6a9-a36dfb628c26"
+					(reference "J17")
+					(unit 1)
+				)
 				(path "/13314f97-080e-4924-a8fe-b4d224920625/a03c39d6-6910-42d9-b21d-b8f6aa6403fb"
 					(reference "J7")
+					(unit 1)
+				)
+				(path "/13314f97-080e-4924-a8fe-b4d224920625/d25a32d7-442e-482e-90f8-47542d85b960"
+					(reference "J16")
 					(unit 1)
 				)
@@
 		(instances
 			(project "standard_puzzle_box"
+				(path "/13314f97-080e-4924-a8fe-b4d224920625/05a99c97-6240-4e5e-b6a9-a36dfb628c26"
+					(reference "#PWR081")
+					(unit 1)
+				)
 				(path "/13314f97-080e-4924-a8fe-b4d224920625/a03c39d6-6910-42d9-b21d-b8f6aa6403fb"
 					(reference "#PWR036")
 					(unit 1)
 				)
+				(path "/13314f97-080e-4924-a8fe-b4d224920625/d25a32d7-442e-482e-90f8-47542d85b960"
+					(reference "#PWR076")
+					(unit 1)
+				)

Commit message: feat: clean up schematic references and run clean annotation
Parts:
- CC_BO1: renamed from C10; footprint (none) -> Capacitor_THT:C_Disc_D5.0mm_W2.5mm_P5.00mm
- CP_BO1: renamed from C11; footprint (none) -> Capacitor_THT:CP_Radial_D10.0mm_P5.00mm
- J_BO1: renamed from J7; value Screw_Terminal_01x02 -> BOOLEAN OUT; footprint (none) -> TerminalBlock_Phoenix:TerminalBlock_Phoenix_MKDS-1,5-2-5.08_1x02_P5.08mm_Horizontal
- R_BO1: renamed from R9; footprint (none) -> Resistor_THT:R_Axial_DIN0411_L9.9mm_D3.6mm_P15.24mm_Horizontal
- R_BO2: renamed from R16; footprint (none) -> Resistor_THT:R_Axial_DIN0411_L9.9mm_D3.6mm_P15.24mm_Horizontal
- renumbered D1flyback2 to D_BO1, Q3 to Q_BO1, U7 to U_BO1
Other:
- moved on the sheet: CC_BO1, CP_BO1

Commit message: fix: run erc and fix errors and warnings
Other:
- note added: "ESP optoisolated boolean output"

Commit message: feat: dump working files before blackout
Parts:
- R_BO1: value 330 Ohm -> 330
- R_BO2: value 10k Ohm -> 10k
Connections:
- net GPIO renamed in
Changed lines of the file:
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@@
-	)
-	(junction
-		(at 104.14 90.17)
-		(diameter 0)
-		(color 0 0 0 0)
 	)
 	(junction
@@
 	(wire
 		(pts
-			(xy 104.14 86.36) (xy 104.14 90.17)
-		)
-		(stroke
-			(width 0)
-			(type default)
-		)
-	)
-	(wire
-		(pts
 			(xy 194.31 82.55) (xy 194.31 99.06)
 		)
@@
 			(width 0)
 			(type default)
-		)
-	)
-	(global_label "GPIO"
-		(shape input)
-		(at 104.14 86.36 90)
-		(fields_autoplaced yes)
-		(effects
-			(font
-				(size 1.27 1.27)
-			)
-			(justify left)
-		)
-		(property "Intersheetrefs" "${INTERSHEET_REFS}"
-			(at 104.14 78.8995 90)
-			(hide yes)
-			(show_name no)
-			(do_not_autoplace no)
-			(effects
-				(font
-					(size 1.27 1.27)
-				)
-				(justify left)
-			)
 		)
 	)
@@
 			)
 		)
-		(property "Value" "330 Ohm"
-			(at 115.57 97.79 0)
+		(property "Value" "330"
+			(at 110.49 97.79 0)
 			(show_name no)
 			(do_not_autoplace no)
@@
 			)
 		)
-		(property "Value" "10k Ohm"
+		(property "Value" "10k"
 			(at 157.48 114.2999 0)
 			(show_name no)

Commit message: feat: salvaging stuff after lossy crash
Parts:
- R_BO1, R_BO2: footprint Resistor_THT:R_Axial_DIN0411_L9.9mm_D3.6mm_P15.24mm_Horizontal -> Resistor_THT:R_Axial_DIN0207_L6.3mm_D2.5mm_P10.16mm_Horizontal
Changed lines of the file:
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@@
 			)
 		)
-		(property "Footprint" "Resistor_THT:R_Axial_DIN0411_L9.9mm_D3.6mm_P15.24mm_Horizontal"
+		(property "Footprint" "Resistor_THT:R_Axial_DIN0207_L6.3mm_D2.5mm_P10.16mm_Horizontal"
 			(at 105.918 96.52 90)
 			(hide yes)
@@
 			)
 		)
-		(property "Footprint" "Resistor_THT:R_Axial_DIN0411_L9.9mm_D3.6mm_P15.24mm_Horizontal"
+		(property "Footprint" "Resistor_THT:R_Axial_DIN0207_L6.3mm_D2.5mm_P10.16mm_Horizontal"
 			(at 156.718 113.03 90)
 			(hide yes)
