File: standard_puzzle_module/signal_output.kicad_sch (KiCad schematic)
At the start: 3 parts, among them J6 Screw_Terminal_01x04

Commit message: chore: clean up
Changed lines of the file:
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@@
 		)
 	)
-	(label "ESP digital signal output (like a speaker module)"
-		(at 115.57 72.39 0)
+	(label "like a speaker module"
+		(at 110.49 69.85 0)
 		(effects
 			(font
+				(size 1.778 1.778)
+			)
+			(justify left bottom)
+		)
+	)
+	(label "ESP digital signal output"
+		(at 110.49 66.04 0)
+		(effects
+			(font

Commit message: feat: unscrew git tracking
Changed lines of the file:
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@@
 		(color 0 0 0 0)
 	)
+	(junction
+		(at 111.76 92.71)
+		(diameter 0)
+		(color 0 0 0 0)
+	)
 	(wire
 		(pts
@@
 		(pts
 			(xy 111.76 88.9) (xy 111.76 92.71)
+		)
+		(stroke
+			(width 0)
+			(type default)
+		)
+	)
+	(wire
+		(pts
+			(xy 107.95 92.71) (xy 111.76 92.71)
 		)
 		(stroke
@@
 				(justify left)
 			)
+		)
+	)
+	(hierarchical_label "out"
+		(shape input)
+		(at 107.95 92.71 180)
+		(effects
+			(font
+				(size 1.27 1.27)
+			)
+			(justify right)
 		)
 	)
@@
 					(unit 1)
 				)
+				(path "/13314f97-080e-4924-a8fe-b4d224920625/d355bcbe-498e-4dcd-b90a-6c2fd2972f51"
+					(reference "#PWR060")
+					(unit 1)
+				)
 			)
 		)
@@
 				(path "/13314f97-080e-4924-a8fe-b4d224920625/87f1a82f-b258-41c3-9586-48c8bc22c59e"
 					(reference "D7")
+					(unit 1)
+				)
+				(path "/13314f97-080e-4924-a8fe-b4d224920625/d355bcbe-498e-4dcd-b90a-6c2fd2972f51"
+					(reference "D15")
 					(unit 1)
 				)
@@
 					(unit 1)
 				)
+				(path "/13314f97-080e-4924-a8fe-b4d224920625/d355bcbe-498e-4dcd-b90a-6c2fd2972f51"
+					(reference "R22")
+					(unit 1)
+				)
 			)
 		)
@@
 					(unit 1)
 				)
+				(path "/13314f97-080e-4924-a8fe-b4d224920625/d355bcbe-498e-4dcd-b90a-6c2fd2972f51"
+					(reference "#PWR027")
+					(unit 1)
+				)
 			)
 		)
@@
 				(path "/13314f97-080e-4924-a8fe-b4d224920625/87f1a82f-b258-41c3-9586-48c8bc22c59e"
 					(reference "#PWR030")
+					(unit 1)
+				)
+				(path "/13314f97-080e-4924-a8fe-b4d224920625/d355bcbe-498e-4dcd-b90a-6c2fd2972f51"
+					(reference "#PWR058")
 					(unit 1)
 				)
@@
 					(unit 1)
 				)
+				(path "/13314f97-080e-4924-a8fe-b4d224920625/d355bcbe-498e-4dcd-b90a-6c2fd2972f51"
+					(reference "J12")
+					(unit 1)
+				)
 			)
 		)
@@
 					(unit 1)
 				)
+				(path "/13314f97-080e-4924-a8fe-b4d224920625/d355bcbe-498e-4dcd-b90a-6c2fd2972f51"
+					(reference "#PWR059")
+					(unit 1)
+				)

Commit message: feat: clean up schematic references and run clean annotation
Parts:
- D_TVSSO1: renamed from D7; value PTVS3V3Z1USK -> P6KE6.8A; footprint Diode_SMD:Nexperia_DSN1608-2_1.6x0.8mm -> Diode_THT:D_DO-15_P12.70mm_Horizontal
- J_SO1: renamed from J6; value Screw_Terminal_01x04 -> SIGNAL OUT; footprint (none) -> TerminalBlock_Phoenix:TerminalBlock_Phoenix_MKDS-1,5-4-5.08_1x04_P5.08mm_Horizontal
- R_SO1: renamed from R15; footprint (none) -> Resistor_THT:R_Axial_DIN0411_L9.9mm_D3.6mm_P15.24mm_Horizontal
Changed lines of the file:
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@@
 					(unit 1)
 				)
-				(path "/13314f97-080e-4924-a8fe-b4d224920625/d355bcbe-498e-4dcd-b90a-6c2fd2972f51"
-					(reference "#PWR060")
+				(path "/13314f97-080e-4924-a8fe-b4d224920625/ab6cca80-8821-447c-8513-efea89d4c4fe"
+					(reference "#PWR018")
 					(unit 1)
 				)
@@
 		(in_pos_files yes)
 		(dnp no)
-		(property "Reference" "D7"
-			(at 134.112 97.028 90)
+		(property "Reference" "D_TVSSO1"
+			(at 125.73 96.52 90)
 			(show_name no)
 			(do_not_autoplace no)
@@
 			)
 		)
-		(property "Value" "PTVS3V3Z1USK"
-			(at 122.428 99.314 90)
+		(property "Value" "P6KE6.8A"
+			(at 125.73 99.06 90)
 			(show_name no)
 			(do_not_autoplace no)
@@
 			)
 		)
-		(property "Footprint" "Diode_SMD:Nexperia_DSN1608-2_1.6x0.8mm"
+		(property "Footprint" "Diode_THT:D_DO-15_P12.70mm_Horizontal"
 			(at 133.985 97.79 0)
 			(hide yes)
@@
 			(project "standard_puzzle_box"
 				(path "/13314f97-080e-4924-a8fe-b4d224920625/87f1a82f-b258-41c3-9586-48c8bc22c59e"
-					(reference "D7")
-					(unit 1)
-				)
-				(path "/13314f97-080e-4924-a8fe-b4d224920625/d355bcbe-498e-4dcd-b90a-6c2fd2972f51"
-					(reference "D15")
+					(reference "D_TVSSO1")
+					(unit 1)
+				)
+				(path "/13314f97-080e-4924-a8fe-b4d224920625/ab6cca80-8821-447c-8513-efea89d4c4fe"
+					(reference "D_TVSSO2")
 					(unit 1)
 				)
@@
 		(dnp no)
 		(fields_autoplaced yes)
-		(property "Reference" "R15"
+		(property "Reference" "R_SO1"
 			(at 129.54 86.36 90)
 			(show_name no)
@@
 			)
 		)
-		(property "Footprint" ""
+		(property "Footprint" "Resistor_THT:R_Axial_DIN0411_L9.9mm_D3.6mm_P15.24mm_Horizontal"
 			(at 129.54 90.932 90)
 			(hide yes)
@@
 			(project "standard_puzzle_box"
 				(path "/13314f97-080e-4924-a8fe-b4d224920625/87f1a82f-b258-41c3-9586-48c8bc22c59e"
-					(reference "R15")
-					(unit 1)
-				)
-				(path "/13314f97-080e-4924-a8fe-b4d224920625/d355bcbe-498e-4dcd-b90a-6c2fd2972f51"
-					(reference "R22")
+					(reference "R_SO1")
+					(unit 1)
+				)
+				(path "/13314f97-080e-4924-a8fe-b4d224920625/ab6cca80-8821-447c-8513-efea89d4c4fe"
+					(reference "R_SO4")
 					(unit 1)
 				)
@@
 					(unit 1)
 				)
-				(path "/13314f97-080e-4924-a8fe-b4d224920625/d355bcbe-498e-4dcd-b90a-6c2fd2972f51"
-					(reference "#PWR027")
+				(path "/13314f97-080e-4924-a8fe-b4d224920625/ab6cca80-8821-447c-8513-efea89d4c4fe"
+					(reference "#PWR015")
 					(unit 1)
 				)
@@
 					(unit 1)
 				)
-				(path "/13314f97-080e-4924-a8fe-b4d224920625/d355bcbe-498e-4dcd-b90a-6c2fd2972f51"
-					(reference "#PWR058")
+				(path "/13314f97-080e-4924-a8fe-b4d224920625/ab6cca80-8821-447c-8513-efea89d4c4fe"
+					(reference "#PWR016")
 					(unit 1)
 				)
@@
 		(dnp no)
 		(fields_autoplaced yes)
-		(property "Reference" "J6"
+		(property "Reference" "J_SO1"
 			(at 162.56 90.1699 0)
 			(show_name no)
@@
 			)
 		)
-		(property "Value" "Screw_Terminal_01x04"
+		(property "Value" "SIGNAL OUT"
 			(at 162.56 92.7099 0)
 			(show_name no)
@@
 			)
 		)
-		(property "Footprint" ""
+		(property "Footprint" "TerminalBlock_Phoenix:TerminalBlock_Phoenix_MKDS-1,5-4-5.08_1x04_P5.08mm_Horizontal"
 			(at 160.02 90.17 0)
 			(hide yes)
@@
 			(project "standard_puzzle_box"
 				(path "/13314f97-080e-4924-a8fe-b4d224920625/87f1a82f-b258-41c3-9586-48c8bc22c59e"
-					(reference "J6")
-					(unit 1)
-				)
-				(path "/13314f97-080e-4924-a8fe-b4d224920625/d355bcbe-498e-4dcd-b90a-6c2fd2972f51"
-					(reference "J12")
+					(reference "J_SO1")
+					(unit 1)
+				)
+				(path "/13314f97-080e-4924-a8fe-b4d224920625/ab6cca80-8821-447c-8513-efea89d4c4fe"
+					(reference "J_SO2")
 					(unit 1)
 				)
@@
 					(unit 1)
 				)
-				(path "/13314f97-080e-4924-a8fe-b4d224920625/d355bcbe-498e-4dcd-b90a-6c2fd2972f51"
-					(reference "#PWR059")
-					(unit 1)
-				)
+				(path "/13314f97-080e-4924-a8fe-b4d224920625/ab6cca80-8821-447c-8513-efea89d4c4fe"
+					(reference "#PWR017")
+					(unit 1)
+				)

Commit message: fix: run erc and fix errors and warnings
Other:
- note added: "Signal output for example, a speaker module"
Changed lines of the file:
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@@
 		(title "ESP digital signal output (like a speaker module)")
+	)
+	(text "Signal output\nfor example, a speaker module\n"
+		(exclude_from_sim no)
+		(at 113.03 68.58 0)
+		(effects
+			(font
+				(size 2.032 2.032)
+				(color 255 97 9 1)
+			)
+			(justify left)
+		)
 	)
 	(junction
@@
 		)
 	)
-	(label "like a speaker module"
-		(at 110.49 69.85 0)
-		(effects
-			(font
-				(size 1.778 1.778)
-			)
-			(justify left bottom)
-		)
-	)
-	(label "ESP digital signal output"
-		(at 110.49 66.04 0)
-		(effects
-			(font
-				(size 1.778 1.778)
-			)
-			(justify left bottom)
-		)
-	)
 	(global_label "GPIO"
 		(shape input)
@@
 		)
 	)
-	(hierarchical_label "out"
+	(hierarchical_label "in"
 		(shape input)
 		(at 107.95 92.71 180)

Commit message: feat: dump working files before blackout
Parts:
- R_SO1: value 100 Ohm -> 100
Connections:
- net GPIO renamed in
Changed lines of the file:
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@@
 		(color 0 0 0 0)
 	)
-	(junction
-		(at 111.76 92.71)
-		(diameter 0)
-		(color 0 0 0 0)
-	)
 	(wire
 		(pts
@@
 	(wire
 		(pts
-			(xy 111.76 92.71) (xy 125.73 92.71)
+			(xy 107.95 92.71) (xy 125.73 92.71)
 		)
 		(stroke
@@
 	(wire
 		(pts
-			(xy 111.76 88.9) (xy 111.76 92.71)
-		)
-		(stroke
-			(width 0)
-			(type default)
-		)
-	)
-	(wire
-		(pts
-			(xy 107.95 92.71) (xy 111.76 92.71)
-		)
-		(stroke
-			(width 0)
-			(type default)
-		)
-	)
-	(wire
-		(pts
 			(xy 146.05 80.01) (xy 146.05 90.17)
 		)
@@
 			(width 0)
 			(type default)
-		)
-	)
-	(global_label "GPIO"
-		(shape input)
-		(at 111.76 88.9 90)
-		(fields_autoplaced yes)
-		(effects
-			(font
-				(size 1.27 1.27)
-			)
-			(justify left)
-		)
-		(property "Intersheetrefs" "${INTERSHEET_REFS}"
-			(at 111.76 81.4395 90)
-			(hide yes)
-			(show_name no)
-			(do_not_autoplace no)
-			(effects
-				(font
-					(size 1.27 1.27)
-				)
-				(justify left)
-			)
 		)
 	)
@@
 			)
 		)
-		(property "Value" "100 Ohm"
+		(property "Value" "100"
 			(at 129.54 88.9 90)
 			(show_name no)

Commit message: feat: salvaging stuff after lossy crash
Parts:
- R_SO1: footprint Resistor_THT:R_Axial_DIN0411_L9.9mm_D3.6mm_P15.24mm_Horizontal -> Resistor_THT:R_Axial_DIN0207_L6.3mm_D2.5mm_P10.16mm_Horizontal
Changed lines of the file:
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@@
 			)
 		)
-		(property "Footprint" "Resistor_THT:R_Axial_DIN0411_L9.9mm_D3.6mm_P15.24mm_Horizontal"
+		(property "Footprint" "Resistor_THT:R_Axial_DIN0207_L6.3mm_D2.5mm_P10.16mm_Horizontal"
 			(at 129.54 90.932 90)
 			(hide yes)
