File: standard_puzzle_module/boolean_input.kicad_sch (KiCad schematic)
At the start: 6 parts

Commit message: feat: improve component placement for pcb
Parts:
- renumbered R_SO2 to R_BI2, R_SO3 to R_BI3
Changed lines of the file:
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@@
 		(dnp no)
 		(fields_autoplaced yes)
-		(property "Reference" "R_SO3"
+		(property "Reference" "R_BI3"
 			(at 160.02 81.2799 0)
 			(show_name no)
@@
 			(project "standard_puzzle_box"
 				(path "/13314f97-080e-4924-a8fe-b4d224920625/3cb740b1-9a02-4adc-be52-b74703d28484"
-					(reference "R_SO10")
+					(reference "R_BI10")
 					(unit 1)
 				)
 				(path "/13314f97-080e-4924-a8fe-b4d224920625/4d21fe22-e137-4b19-b5e5-b3ac06ec1179"
-					(reference "R_SO8")
+					(reference "R_BI8")
 					(unit 1)
 				)
 				(path "/13314f97-080e-4924-a8fe-b4d224920625/5f64ce72-3807-4d88-a28a-0ca03d044e7a"
-					(reference "R_SO3")
+					(reference "R_BI3")
 					(unit 1)
 				)
 				(path "/13314f97-080e-4924-a8fe-b4d224920625/a53fbb5d-1a9d-4dfa-ba02-9f03c2e38d67"
-					(reference "R_SO6")
+					(reference "R_BI6")
 					(unit 1)
 				)
@@
 		(dnp no)
 		(fields_autoplaced yes)
-		(property "Reference" "R_SO2"
+		(property "Reference" "R_BI2"
 			(at 128.27 87.6299 0)
 			(show_name no)
@@
 			(project "standard_puzzle_box"
 				(path "/13314f97-080e-4924-a8fe-b4d224920625/3cb740b1-9a02-4adc-be52-b74703d28484"
-					(reference "R_SO9")
+					(reference "R_BI9")
 					(unit 1)
 				)
 				(path "/13314f97-080e-4924-a8fe-b4d224920625/4d21fe22-e137-4b19-b5e5-b3ac06ec1179"
-					(reference "R_SO7")
+					(reference "R_BI7")
 					(unit 1)
 				)
 				(path "/13314f97-080e-4924-a8fe-b4d224920625/5f64ce72-3807-4d88-a28a-0ca03d044e7a"
-					(reference "R_SO2")
+					(reference "R_BI2")
 					(unit 1)
 				)
 				(path "/13314f97-080e-4924-a8fe-b4d224920625/a53fbb5d-1a9d-4dfa-ba02-9f03c2e38d67"
-					(reference "R_SO5")
-					(unit 1)
-				)
+					(reference "R_BI5")
+					(unit 1)
+				)
