File: standard_puzzle_module/_restore_backup_2026-08-24T23-28-08-749/standard_puzzle_box.kicad_pcb (KiCad board)
At the start: 2 copper layers, 76 parts, among them U1 ESP32-C3-DevKitM-1

Commit message: feat: draft component placement for pcb
Parts:
- R_BO1, R_BO2, R_BO3, R_BO4, R_BO5, R_BO6, R_SIN1, R_SIN2, R_SIN3, R_SIN4, R_SO1, R_SO10, R_SO2, R_SO3, R_SO4, R_SO5, R_SO6, R_SO7, R_SO8, R_SO9: footprint Resistor_THT:R_Axial_DIN0411_L9.9mm_D3.6mm_P15.24mm_Horizontal -> Resistor_THT:R_Axial_DIN0207_L6.3mm_D2.5mm_P10.16mm_Horizontal
- moved R_BO6 204.4 mm to (106.4, 87.4)
- moved J_BI4 197.0 mm to (172.0, 32.2), turned to 180 degrees
- moved J_BI3 190.6 mm to (188.6, 31.8), turned to 180 degrees
- moved CP_BO2 188.4 mm to (153.9, 106.0)
- moved R_BO4 187.1 mm to (139.2, 86.6)
- moved R_BO5 184.8 mm to (131.7, 93.8), turned to -90 degrees
- moved D_BO2 183.9 mm to (153.8, 98.5), turned to 180 degrees
- moved J_BO2 183.1 mm to (146.9, 106.0), turned to 180 degrees
- moved CP_BO1 181.5 mm to (184.1, 105.7)
- moved U_BO2 181.4 mm to (165.2, 88.6), turned to 180 degrees
- moved Q_BO2 179.6 mm to (146.2, 91.5), turned to 180 degrees
- moved D_BI3 179.6 mm to (191.0, 50.1), turned to 180 degrees
- moved D_BI4 179.5 mm to (177.5, 50.1), turned to 180 degrees
- moved U_BI4 177.8 mm to (174.0, 56.6), turned to 180 degrees
- moved CC_BO2 177.5 mm to (158.8, 92.9), turned to 180 degrees
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Routing:
- net +12V: track 8.02 -> 85.9 mm
- net GND: track 57.0 -> 93.4 mm, vias 8 -> 14
- net +5V: track 43.5 -> 10.6 mm
- net +3.3V: track 29.4 -> 0.00 mm, vias 0 -> 1
- net Net-(D_BO3-A): track 0.00 -> 15.9 mm
- net Net-(D_BO1-A): track 0.00 -> 15.9 mm
- net Net-(D_BO2-A): track 0.00 -> 15.2 mm
- net Net-(Q_BO3-G): track 0.00 -> 14.2 mm
- net Net-(Q_BO2-G): track 0.00 -> 13.7 mm
- net Net-(R_BO5-Pad1): track 0.00 -> 13.7 mm, vias 0 -> 2
- net /signal_input/out: track 13.3 -> 0.00 mm
- net Net-(R_BO3-Pad1): track 0.00 -> 11.9 mm, vias 0 -> 2
- net Net-(Q_BO1-G): track 0.00 -> 11.7 mm
- net Net-(R_BO1-Pad1): track 0.00 -> 11.6 mm, vias 0 -> 2
- net Net-(J_BI1-Pin_2): track 8.05 -> 0.00 mm
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