File: universal_puzzle_node/universal_puzzle_node.kicad_pcb (KiCad board)
At the start: 2 copper layers, 97.2 x 91 mm, 77 parts, among them U1 ESP32-C3-SuperMini

Commit message: chore: rename to universal puzzle node everywhere
Other:
- board text added: "One must imagine Sisyphus happy."
- board text added: "commit sha: b99e2af"
Changed lines of the file:
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@@
 		(capping no)
 		(filling no)
-		(zone_defaults)
 		(grid_origin 29 155.5)
 		(pcbplotparams
@@
 		)
 	)
+	(gr_text "One must imagine Sisyphus happy."
+		(at 136.95 55.45 0)
+		(layer "B.SilkS")
+		(effects
+			(font
+				(size 1 1)
+				(thickness 0.1)
+			)
+			(justify left bottom mirror)
+		)
+	)
+	(gr_text "commit sha: b99e2af"
+		(at 136.95 58.95 0)
+		(layer "B.SilkS")
+		(effects
+			(font
+				(size 1 1)
+				(thickness 0.1)
+			)
+			(justify left bottom mirror)
+		)
+	)
 	(gr_text "Licensed under CC-BY-SA 4.0"
 		(at 137 60.45 0)
@@
 	)
 	(segment
-		(start 143.8 31)
-		(end 148.7 35.9)
+		(start 118.8 37.38)
+		(end 126.37 37.38)
 		(width 0.25)
 		(layer "F.Cu")
@@
 	)
 	(segment
-		(start 118.8 37.38)
-		(end 126.37 37.38)
+		(start 126.37 37.38)
+		(end 132.7 31.05)
 		(width 0.25)
 		(layer "F.Cu")
@@
 	)
 	(segment
-		(start 132.75 31)
-		(end 143.8 31)
+		(start 148.7 35.9)
+		(end 152.15 35.9)
 		(width 0.25)
 		(layer "F.Cu")
@@
 	)
 	(segment
-		(start 126.37 37.38)
-		(end 132.75 31)
+		(start 143.85 31.05)
+		(end 148.7 35.9)
 		(width 0.25)
 		(layer "F.Cu")
@@
 	)
 	(segment
-		(start 148.7 35.9)
-		(end 152.15 35.9)
+		(start 132.7 31.05)
+		(end 143.85 31.05)
 		(width 0.25)
 		(layer "F.Cu")
@@
 	)
 	(segment
-		(start 133 28.7)
+		(start 152.09 28.5)
 		(end 152.29 28.7)
 		(width 0.25)
@@
 	(segment
 		(start 126.86 34.84)
-		(end 133 28.7)
+		(end 133.2 28.5)
+		(width 0.25)
+		(layer "F.Cu")
+		(net "/signal_output/in")
+	)
+	(segment
+		(start 133.2 28.5)
+		(end 152.09 28.5)
 		(width 0.25)
 		(layer "F.Cu")

Commit message: build: add gerber files with previous commit SHA
Other:
- board text added: "commit sha: ecc5202"
- board text removed: "commit sha: b99e2af"
Changed lines of the file:
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@@
 		)
 	)
-	(gr_text "commit sha: b99e2af"
+	(gr_text "commit sha: ecc5202"
 		(at 136.95 58.95 0)
 		(layer "B.SilkS")
